File: hardware/esp32-c3-sensor-board-rev2.kicad_pcb (KiCad board)
At the start: 2 copper layers, 46 x 89 mm, 14 parts, among them J1 BME280_Module, J2 BH1750_Module, J3 Relay, J4 Button, J5 BREAKOUT, U1 ESP32-C3-SuperMini, U2 HLK-LD2410C

Commit message: Fit J5 as a standard 1x14 female socket
Replace the bare breakout_1x14 footprint with the standard
Connector_PinSocket_2.54mm:PinSocket_1x14_P2.54mm_Vertical at the same
position (40, 25). Pad positions, drills and nets are unchanged; pad 1 is
now the standard rectangular pin-1 marker and the socket has a 3D model.

- Update the schematic J5 Footprint field so a future F8 keeps the socket.
- Update the JLC BOM footprint row and all docs/QUOTE wording (J5 is now a
  fitted socket, not bare holes).
- Refill zones and re-run DRC: 0 errors / 0 unconnected (2 cosmetic silk
  warnings).
- Regenerate gerbers, drill, job file and gerber zip from the final board.

Co-Authored-By: Claude Code <noreply@anthropic.com>
Parts:
- J5: footprint sensor-board:breakout_1x14 -> Connector_PinSocket_2.54mm:PinSocket_1x14_P2.54mm_Vertical

Commit message: Add JP1/JP2/JP3 pin-number labels on the bottom silkscreen
The jumper pins had no visible numbering. Add mirrored 1-3 numbers next to
each column on B.Silk (1-2 for JP3) and the JP1/JP2/JP3 column names below
them. The bottom is where the shunts are fitted and is not covered by the
BME280 module.

Remove the large B.Silk jumper boxes to make room for the numbers; the short
1-2 default-pair ticks remain. The front JP1/JP2/JP3 and CSB/SDO/ADDR labels
are unchanged.

Update README and docs/pinout with the pin-numbering note. Regenerate gerbers,
drill, job file and zip. DRC 0 errors / 0 unconnected (2 cosmetic silk
warnings).

Co-Authored-By: Claude Code <noreply@anthropic.com>
Other:
- board text added: "1"
- board text added: "2"
- board text added: "3"
Changed lines of the file:
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@@
-	)
-	(gr_line
-		(start 1.9 49.4)
-		(end 5.1 49.4)
-		(stroke
-			(width 0.12)
-			(type default)
-		)
-		(layer "B.SilkS")
-	)
-	(gr_line
-		(start 1.9 58)
-		(end 1.9 49.4)
-		(stroke
-			(width 0.12)
-			(type default)
-		)
-		(layer "B.SilkS")
 	)
 	(gr_line
@@
 	)
 	(gr_line
-		(start 5.1 49.4)
-		(end 5.1 58)
-		(stroke
-			(width 0.12)
-			(type default)
-		)
-		(layer "B.SilkS")
-	)
-	(gr_line
-		(start 5.1 58)
-		(end 1.9 58)
-		(stroke
-			(width 0.12)
-			(type default)
-		)
-		(layer "B.SilkS")
-	)
-	(gr_line
-		(start 5.5 49.4)
-		(end 8.7 49.4)
-		(stroke
-			(width 0.12)
-			(type default)
-		)
-		(layer "B.SilkS")
-	)
-	(gr_line
-		(start 5.5 58)
-		(end 5.5 49.4)
-		(stroke
-			(width 0.12)
-			(type default)
-		)
-		(layer "B.SilkS")
-	)
-	(gr_line
 		(start 6.3 52.47)
 		(end 7.9 52.47)
@@
 	)
 	(gr_line
-		(start 8.7 49.4)
-		(end 8.7 58)
-		(stroke
-			(width 0.12)
-			(type default)
-		)
-		(layer "B.SilkS")
-	)
-	(gr_line
-		(start 8.7 58)
-		(end 5.5 58)
-		(stroke
-			(width 0.12)
-			(type default)
-		)
-		(layer "B.SilkS")
-	)
-	(gr_line
-		(start 9.1 49.4)
-		(end 12.3 49.4)
-		(stroke
-			(width 0.12)
-			(type default)
-		)
-		(layer "B.SilkS")
-	)
-	(gr_line
-		(start 9.1 55.3)
-		(end 9.1 49.4)
-		(stroke
-			(width 0.12)
-			(type default)
-		)
-		(layer "B.SilkS")
-	)
-	(gr_line
 		(start 9.9 52.47)
 		(end 11.5 52.47)
 		(stroke
 			(width 0.3)
-			(type default)
-		)
-		(layer "B.SilkS")
-	)
-	(gr_line
-		(start 12.3 49.4)
-		(end 12.3 55.3)
-		(stroke
-			(width 0.12)
-			(type default)
-		)
-		(layer "B.SilkS")
-	)
-	(gr_line
-		(start 12.3 55.3)
-		(end 9.1 55.3)
-		(stroke
-			(width 0.12)
 			(type default)
 		)
@@
 		)
 	)
+	(gr_text "1"
+		(at 1.8 51.2 0)
+		(layer "B.SilkS")
+		(effects
+			(font
+				(size 0.8 0.8)
+				(thickness 0.12)
+			)
+			(justify mirror)
+		)
+	)
+	(gr_text "2"
+		(at 1.8 53.74 0)
+		(layer "B.SilkS")
+		(effects
+			(font
+				(size 0.8 0.8)
+				(thickness 0.12)
+			)
+			(justify mirror)
+		)
+	)
+	(gr_text "3"
+		(at 1.8 56.28 0)
+		(layer "B.SilkS")
+		(effects
+			(font
+				(size 0.8 0.8)
+				(thickness 0.12)
+			)
+			(justify mirror)
+		)
+	)
+	(gr_text "JP1"
+		(at 1.8 58.6 0)
+		(layer "B.SilkS")
+		(effects
+			(font
+				(size 0.8 0.8)
+				(thickness 0.12)
+			)
+			(justify mirror)
+		)
+	)
+	(gr_text "1"
+		(at 5.4 51.2 0)
+		(layer "B.SilkS")
+		(effects
+			(font
+				(size 0.8 0.8)
+				(thickness 0.12)
+			)
+			(justify mirror)
+		)
+	)
+	(gr_text "2"
+		(at 5.4 53.74 0)
+		(layer "B.SilkS")
+		(effects
+			(font
+				(size 0.8 0.8)
+				(thickness 0.12)
+			)
+			(justify mirror)
+		)
+	)
+	(gr_text "3"
+		(at 5.4 56.28 0)
+		(layer "B.SilkS")
+		(effects
+			(font
+				(size 0.8 0.8)
+				(thickness 0.12)
+			)
+			(justify mirror)
+		)
+	)
+	(gr_text "JP2"
+		(at 5.4 58.6 0)
+		(layer "B.SilkS")
+		(effects
+			(font
+				(size 0.8 0.8)
+				(thickness 0.12)
+			)
+			(justify mirror)
+		)
+	)
+	(gr_text "1"
+		(at 9 51.2 0)
+		(layer "B.SilkS")
+		(effects
+			(font
+				(size 0.8 0.8)
+				(thickness 0.12)
+			)
+			(justify mirror)
+		)
+	)
+	(gr_text "2"
+		(at 9 53.74 0)
+		(layer "B.SilkS")
+		(effects
+			(font
+				(size 0.8 0.8)
+				(thickness 0.12)
+			)
+			(justify mirror)
+		)
+	)
+	(gr_text "JP3"
+		(at 9 58.6 0)
+		(layer "B.SilkS")
+		(effects
+			(font
+				(size 0.8 0.8)
+				(thickness 0.12)
+			)
+			(justify mirror)
+		)
+	)
